File: stendas/stendas.kicad_pcb (KiCad board)
At the start: 2 copper layers, 138 x 81 mm, 69 parts, among them J1 RA8875, J17 MB SLAVE, J2 EXT1, J22 MB MASTER, J3 EXT2, J5 EXT, J6 Service, M1 STM32F4-Disco, Q1 BC817, U1 ST485B, U2 ST485B

Commit message: pirma plokstes versija
Parts:
- removed the ? at (141.0, 100.0)
- removed the ? at (141.0, 108.6)
- added ?: , Connector_Pin:Pin_D0.7mm_L6.5mm_W1.8mm_FlatFork, F.Cu at (140.7, 116.5)
- added ?: , Connector_Pin:Pin_D0.7mm_L6.5mm_W1.8mm_FlatFork, F.Cu at (140.8, 108.6)
- added ?: , Connector_Pin:Pin_D0.7mm_L6.5mm_W1.8mm_FlatFork, F.Cu at (140.7, 125.7)
- added ?: , Connector_Pin:Pin_D0.7mm_L6.5mm_W1.8mm_FlatFork, F.Cu at (140.8, 100.0)
- added C2: 0.1, Capacitor_SMD:C_0805_2012Metric, F.Cu at (134.4, 83.4)
- added C21: 0.1, Capacitor_SMD:C_0805_2012Metric, F.Cu at (157.2, 134.2)
- added R13: 4.7k, Resistor_SMD:R_0805_2012Metric, F.Cu at (151.5, 114.5)
- added R14: 4.7k, Resistor_SMD:R_0805_2012Metric, F.Cu at (151.5, 112.5)
- added U3: 24LC32, Package_SO:SOIC-8_3.9x4.9mm_P1.27mm, F.Cu at (145.8, 112.3)
- moved C3 5.77 mm to (153.0, 120.3)
- moved C6 4.47 mm to (144.7, 119.8)
- moved C19 2.80 mm to (156.0, 124.8)
- moved C4 2.57 mm to (137.6, 120.3)
- renumbered C2 to C1, C12 to C11, C1 to C15, C11 to C16, C15 to C17, C16 to C18, C17 to C19, C18 to C20, C19 to C22, J17 to J1, J22 to J2, J1 to J3, J3 to J4, J2 to J7, R6 to R2, R2 to R3, R3 to R4, R7 to R5, R8 to R6, R4 to R7, R9 to R8, R5 to R9
Connections:
- net Net-(M1-Pad10) renamed /ADC_CH12
- net Net-(M1-Pad13) renamed /ADC_CH3
- net Net-(M1-Pad14) renamed /ADC_CH2
- net Net-(M1-Pad19) renamed /ADC_CH15
- net Net-(M1-Pad20) renamed /ADC_CH14
- net Net-(M1-Pad21) renamed /ADC_CH9
- net Net-(M1-Pad22) renamed /ADC_CH8
- net Net-(M1-Pad69) renamed /BUZ
- net Net-(M1-Pad7) renamed /ADC_CH11
- net Net-(M1-Pad8) renamed /ADC_CH10
- net Net-(M1-Pad89) renamed /SWDCLK
- net Net-(M1-Pad9) renamed /ADC_CH13
- net Net-(M1-Pad90) renamed /TEST_OUT
- net Net-(M1-Pad92) renamed /SWDIO
- DE pad 1: /DE -> /U4DE
- J7 pad 10: Net-(J2-Pad10) -> /PWM3
- J7 pad 11: Net-(J2-Pad11) -> /DS_DATA
- J7 pad 16: Net-(J2-Pad16) -> /SCL
- J7 pad 17: Net-(J2-Pad17) -> /SDA
- J7 pad 7: Net-(J2-Pad7) -> /PWM2
- J7 pad 8: Net-(J2-Pad8) -> /PWM1
- J7 pad 9: Net-(J2-Pad9) -> /PWM4
- M1 pad 24: Net-(M1-Pad24) -> /U4DE
- M1 pad 3: Net-(M1-Pad3) -> /VDD
- M1 pad 4: Net-(M1-Pad4) -> /VDD
- M1 pad 73: Net-(M1-Pad73) -> /SCL
- M1 pad 74: Net-(M1-Pad74) -> /SDA
- M1 pad 81: Net-(M1-Pad81) -> /U5DE
- M1 pad 88: Net-(M1-Pad88) -> /DS_DATA
- M1 pad 95: Net-(M1-Pad95) -> /PWM3
- M1 pad 96: Net-(M1-Pad96) -> /PWM4
- M1 pad 97: Net-(M1-Pad97) -> /PWM1
- M1 pad 98: Net-(M1-Pad98) -> /PWM2
Routing:
- net /3VDC: track 152.1 -> 187.3 mm
- net /SDA: track 0.00 -> 33.8 mm
- net /SCL: track 0.00 -> 32.9 mm
- net GND: track 65.7 -> 74.9 mm
- net /VDD: track 0.00 -> 5.16 mm
- net /U4DE: track 0.00 -> 4.01 mm
- net /DE: track 4.01 -> 0.00 mm
- net Net-(C21-Pad2): track 0.00 -> 2.60 mm

Commit message: remapinti pinai - plokste pritaikyta darbui su sd-card
Connections:
- net /LD7 renamed Net-(M1-Pad94)
- net Net-(M1-Pad87) renamed /SDIO_D2
- J7 pad 10: /PWM3 -> /PWM1
- J7 pad 25: Net-(J7-Pad25) -> /ADC_CH8
- J7 pad 26: Net-(J7-Pad26) -> /ADC_CH9
- J7 pad 27: Net-(J7-Pad27) -> /ADC_CH10
- J7 pad 28: Net-(J7-Pad28) -> /ADC_CH11
- J7 pad 29: Net-(J7-Pad29) -> /ADC_CH12
- J7 pad 30: Net-(J7-Pad30) -> /ADC_CH13
- J7 pad 31: Net-(J7-Pad31) -> /ADC_CH14
- J7 pad 32: Net-(J7-Pad32) -> /ADC_CH15
- J7 pad 7: /PWM2 -> /PWM4
- J7 pad 8: /PWM1 -> /PWM3
- J7 pad 9: /PWM4 -> /PWM2
- M1 pad 13: /ADC_CH3 -> /U2RX
- M1 pad 14: /ADC_CH2 -> /U2TX
- M1 pad 19: /ADC_CH15 -> /ADC_CH11
- M1 pad 20: /ADC_CH14 -> /ADC_CH10
- M1 pad 38: Net-(M1-Pad38) -> /PWM3
- M1 pad 39: Net-(M1-Pad39) -> /PWM4
- M1 pad 61: Net-(M1-Pad61) -> /PWM2
- M1 pad 64: Net-(M1-Pad64) -> /PWM1
- M1 pad 69: /BUZ -> /BUZZ
- M1 pad 7: /ADC_CH11 -> /ADC_CH15
- M1 pad 8: /ADC_CH10 -> /ADC_CH14
- M1 pad 81: /U5DE -> /U2DE
- M1 pad 84: /U5RX -> /SDIO_CMD
- M1 pad 85: /U5TX -> /SDIO_CK
- M1 pad 88: /DS_DATA -> /SDIO_D3
- M1 pad 95: /PWM3 -> /SDIO_D0
- M1 pad 96: /PWM4 -> /SDIO_D1
- M1 pad 97: /PWM1 -> /SD_DETECT
- M1 pad 98: /PWM2 -> Net-(M1-Pad98)
- U2 pad 1: /U5RX -> /U2RX
- U2 pad 2: /U5DE -> /U2DE
- U2 pad 3: /U5DE -> /U2DE
- U2 pad 4: /U5TX -> /U2TX
